Commit message: Changes in simulation file

File: Quadruped_Robot_Sim/description/quadruped_robot.urdf (robot description, URDF)
Before this commit: robot quadruped_robot, 9 links, 8 joints
Joints:
- joint bottom_bl: limit lower=-3.14 upper=3.14 effort=100 velocity=0.1 -> lower=-1.57 upper=1.57 effort=100 velocity=10
- joint bottom_br: limit lower=-3.14 upper=3.14 effort=100 velocity=0.1 -> lower=-1.57 upper=1.57 effort=100 velocity=10
- joint bottom_fl: limit lower=-3.14 upper=3.14 effort=100 velocity=0.1 -> lower=-1.57 upper=1.57 effort=100 velocity=10
- joint bottom_fr: limit lower=-3.14 upper=3.14 effort=100 velocity=0.1 -> lower=-1.57 upper=1.57 effort=100 velocity=10
- joint up_bl: limit lower=-3.14 upper=3.14 effort=100 velocity=0.1 -> lower=-1.57 upper=1.57 effort=100 velocity=10
- joint up_br: limit lower=-3.14 upper=3.14 effort=100 velocity=0.1 -> lower=-1.57 upper=1.57 effort=100 velocity=10
- joint up_fl: limit lower=-3.14 upper=3.14 effort=100 velocity=0.1 -> lower=-1.57 upper=1.57 effort=100 velocity=10
- joint up_fr: limit lower=-3.14 upper=3.14 effort=100 velocity=0.1 -> lower=-1.57 upper=1.57 effort=100 velocity=10

File: Quadruped_Robot_Sim/description/quadruped_robot.xacro (robot description, xacro)
@@ -7,6 +7,6 @@
 	<xacro:include filename="inertias.xacro"/>
 	<!-- Property Definition -->
-	<xacro:property name="joint_limit_low" value="-3.14"/>
-	<xacro:property name="joint_limit_up" value="3.14"/>
+	<xacro:property name="joint_limit_low" value="-1.57"/>
+	<xacro:property name="joint_limit_up" value="1.57"/>
 	<!-- Macros for Links and Joints -->
 	<xacro:macro name="create_link" params="name base_size x y z material:=grey">
@@ -36,6 +36,6 @@
 			<origin xyz="${x} ${y} ${z}"/>
 			<axis xyz="0 -1 0"/>
-			<limit lower="${joint_limit_low}" upper="${joint_limit_up}" effort="100" velocity="0.1"/>
-			<dynamics damping="0.1" friction="0.1"/>
+			<limit lower="${joint_limit_low}" upper="${joint_limit_up}" effort="100" velocity="10"/>
+			<dynamics damping="1" friction="0.01"/>
 		</joint>
 	</xacro:macro>

File: Quadruped_Robot_Sim/simulation/models/quadruped_robot_fixed/quadruped_robot_fixed.urdf (robot description, URDF)
Before this commit: robot quadruped_robot_fixed, 10 links, 9 joints
Joints:
- joint bottom_bl: limit lower=-3.14 upper=3.14 effort=100 velocity=0.1 -> lower=-1.57 upper=1.57 effort=100 velocity=10
- joint bottom_br: limit lower=-3.14 upper=3.14 effort=100 velocity=0.1 -> lower=-1.57 upper=1.57 effort=100 velocity=10
- joint bottom_fl: limit lower=-3.14 upper=3.14 effort=100 velocity=0.1 -> lower=-1.57 upper=1.57 effort=100 velocity=10
- joint bottom_fr: limit lower=-3.14 upper=3.14 effort=100 velocity=0.1 -> lower=-1.57 upper=1.57 effort=100 velocity=10
- joint up_bl: limit lower=-3.14 upper=3.14 effort=100 velocity=0.1 -> lower=-1.57 upper=1.57 effort=100 velocity=10
- joint up_br: limit lower=-3.14 upper=3.14 effort=100 velocity=0.1 -> lower=-1.57 upper=1.57 effort=100 velocity=10
- joint up_fl: limit lower=-3.14 upper=3.14 effort=100 velocity=0.1 -> lower=-1.57 upper=1.57 effort=100 velocity=10
- joint up_fr: limit lower=-3.14 upper=3.14 effort=100 velocity=0.1 -> lower=-1.57 upper=1.57 effort=100 velocity=10
